File: atmel.kicad_pcb (KiCad board)
At the start: 2 copper layers, 29.6 x 25.4 mm, 9 parts, among them J1 Güç Girişi, U1 NCP1117-5.0_SOT223, U2 ATmega328P-AU, Y1 16MHz

Commit message: 21 Mart Ev
Parts:
- added J2: ICSP, Connector_PinHeader_1.27mm:PinHeader_2x03_P1.27mm_Vertical, F.Cu at (129.5, 38.1)
- added J3: Reset Jmp, Connector_PinHeader_1.27mm:PinHeader_1x02_P1.27mm_Vertical, F.Cu at (133.3, 36.8)
- added R1: 10K, Resistor_SMD:R_0603_1608Metric_Pad1.05x0.95mm_HandSolder, F.Cu at (133.3, 40.6)
Connections:
- U2 pad 15: Net-(U2-Pad15) -> MOSI
- U2 pad 16: Net-(U2-Pad16) -> MISO
- U2 pad 17: Net-(U2-Pad17) -> SCK
- U2 pad 29: Net-(U2-Pad29) -> RESET
Routing:
- net RESET: track 0.00 -> 23.2 mm
- net MOSI: track 0.00 -> 15.4 mm, vias 0 -> 1
- net SCK: track 0.00 -> 13.8 mm, vias 0 -> 1
- net +5V: track 60.5 -> 72.4 mm
- net MISO: track 0.00 -> 11.3 mm, vias 0 -> 1
- net GND: track 14.0 -> 8.83 mm, vias 0 -> 1
- added copper zone on B.Cu, net GND
Other:
- board size 29.6 x 25.4 mm -> 38.8 x 25.4 mm
